File: hardware/2003-hall-sensors-board-platter/2003-hall-sensors-board-platter.kicad_pcb (KiCad board)
At the start: 2 copper layers, 72 x 20 mm, 9 parts, among them J1 Conn_01x04_Male, U1 SS49X, U2 SS49X

Commit message: updated License
Other:
- board text added: "Licensed under CERN-OHL-S v2"
- board text removed: "Licensed under CERN-OHL-P v2"
Changed lines of the file:
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@@
   (page A4)
   (layers
-    (0 F.Cu signal)
-    (31 B.Cu signal)
+    (0 F.Cu signal hide)
+    (31 B.Cu signal hide)
     (32 B.Adhes user hide)
     (33 F.Adhes user hide)
@@
     )
   )
-  (gr_text "Licensed under\nCERN-OHL-P v2" (at 155.25 103.75 90) (layer B.SilkS)
+  (gr_text "Licensed under\nCERN-OHL-S v2" (at 155.25 103.75 90) (layer B.SilkS)
     (effects (font (size 0.75 0.75) (thickness 0.125)) (justify mirror))
   )
